File: BatteryMonitorModule.kicad_sch (KiCad schematic)
At the start: 86 parts, among them K1 G5LE-1, Q1 AO3401A, Q2 MMBT2222A, Q3 IRFZ44NPBF, Q3_DRV MMBT2222A, Q4 IRLML2502TRPBF, U1 STM32G0B1CCT6, U3 AP63203WU-7, U4 MIC5219-3.3YM5-TR, U5 AP63205WU-7

Commit message: assigned mfg part numbers
Parts:
- added LED? (x3): WS2812B 5mm TH, LED_THT:LED_D5.0mm, symbol LED:WS2812B
- F?: renamed from F3; footprint Fuse:Fuse_Blade_ATM_Mini -> (none)
- F?: renamed from F2; footprint Fuse:Fuse_Blade_ATM_Mini -> (none)
- F?: renamed from F1; footprint Fuse:Fuse_Blade_ATM_Mini -> (none)
- R_BLEED?: renamed from R_BLEED1; footprint Resistor_THT:R_Axial_DIN0516_L15.5mm_D5.3mm_P22.86mm_Horizontal -> Resistor_THT:R_Axial_DIN0516_L15.5mm_D5.3mm_P20.32mm_Horizontal
- R_BLEED?: renamed from R_BLEED2; footprint Resistor_THT:R_Axial_DIN0516_L15.5mm_D5.3mm_P22.86mm_Horizontal -> Resistor_THT:R_Axial_DIN0516_L15.5mm_D5.3mm_P20.32mm_Horizontal
- renumbered C_12V_IN to C_12V_IN?, C_5V_IN to C_5V_IN?, C_5V_OUT to C_5V_OUT?, C_BST to C_BST?, C_BST2 to C_BST?, C_BULK_3V3 to C_BULK_3V?, C_IN to C_IN?, C_INA_VS to C_INA_VS?, C_NRST to C_NRST?, C_OUT to C_OUT?, C_U4_IN to C_U4_IN?, C_U4_OUT to C_U4_OUT?, C_VBAT to C_VBAT?, C_VDD2 to C_VDD?, C_VDD1 to C_VDD?, C_VDDIO2 to C_VDDIO?, C_VDD_BULK to C_VDD_BULK?, C_VREF to C_VREF?, D1 to D?, D_12V to D_12V?, D_FAN to D_FAN?, D_USB to D_USB?, FB1 to FB?, FH1 to FH?, FH3 to FH?, FH2 to FH?, J_DISP_I2C to J_DISP_I2C?, J_DISP_SPI to J_DISP_SPI?, J_EXP_A to J_EXP_A?, J_EXP_B to J_EXP_B?, J_FAN to J_FAN?, J_FAN_SEL to J_FAN_SEL?, J_LED to J_LED?, J_NFC to J_NFC?, J_PWR_A to J_PWR_A?, J_PWR_B to J_PWR_B?, J_SW1 to J_SW?, J_SW3 to J_SW?, J_SW2 to J_SW?, J_SWD to J_SWD?, J_UART to J_UART?, J_USB to J_USB?, K1 to K?, L2 to L?, L1 to L?, LED_DBG1 to LED_DBG?, LED_DBG2 to LED_DBG?, Q3_DRV to Q3_DRV?, Q3 to Q?, Q2 to Q?, Q4 to Q?, Q1 to Q?, RT1 to RT?, R_12V_H to R_12V_H?, R_12V_L to R_12V_L?, R_B3 to R_B?, R_BAT_H to R_BAT_H?, R_BAT_L to R_BAT_L?, R_BOOT0 to R_BOOT?, R_BOOT_G3 to R_BOOT_G?, R_CC1 to R_CC?, R_CC2 to R_CC?, R_CHG_H to R_CHG_H?, R_CHG_L to R_CHG_L?, R_FAN_G to R_FAN_G?, R_FAN_PD to R_FAN_PD?, R_G1 to R_G?, R_G3 to R_G?, R_GATE_K1 to R_GATE_K?, R_I2C1_SCL to R_I2C1_SCL?, R_I2C1_SDA to R_I2C1_SDA?, R_LED_DIN to R_LED_DIN?, R_NTC_S to R_NTC_S?, R_PG to R_PG?, R_SHUNT to R_SHUNT?, SW_BOOT to SW_BOOT?, SW_RST to SW_RST?, U1 to U?, U4 to U?, U5 to U?, U3 to U?

Commit message: Revert "assigned mfg part numbers"
This reverts commit d05d25c7e7cb63e1a29fd6f965ec26ad4da439bc.
Parts:
- removed LED? (x3): WS2812B 5mm TH, LED_THT:LED_D5.0mm, symbol LED:WS2812B
- F1, F2, F3: renamed from F?; footprint (none) -> Fuse:Fuse_Blade_ATM_Mini
- R_BLEED1, R_BLEED2: renamed from R_BLEED?; footprint Resistor_THT:R_Axial_DIN0516_L15.5mm_D5.3mm_P20.32mm_Horizontal -> Resistor_THT:R_Axial_DIN0516_L15.5mm_D5.3mm_P22.86mm_Horizontal
- gave numbers to parts that had none: 81
