File: BatteryMonitorModule.kicad_sch (KiCad schematic)
At the start: 86 parts, among them K1 G5LE-1, Q1 AO3401A, Q2 MMBT2222A, Q3 IRFZ44NPBF, Q3_DRV MMBT2222A, Q4 IRLML2502TRPBF, U1 STM32G0B1CCT6, U3 AP63203WU-7, U4 MIC5219-3.3YM5-TR, U5 AP63205WU-7

Commit message: assigned mfg part numbers
Co-Authored-By: Claude Opus 4.6 (1M context) <noreply@anthropic.com>
Parts:
- C_12V_IN, C_5V_IN, C_IN: DK_PN (none) -> 1276-6470-1-ND; MPN (none) -> CL21A106KAYNNNE
- C_5V_OUT, C_OUT: DK_PN (none) -> 1276-6471-1-ND; MPN (none) -> CL21A226MAQNNNE
- C_BST, C_BST2: DK_PN (none) -> 1276-1946-1-ND; MPN (none) -> CL05B104KO5NNNC
- C_BULK_3V3, C_VDD_BULK: DK_PN (none) -> 1276-6474-1-ND; MPN (none) -> CL21A475KAQNNNE
- C_INA_VS, C_NRST, C_VBAT, C_VDD1, C_VDD2, C_VDDIO2, C_VREF: DK_PN (none) -> 1276-1931-1-ND; MPN (none) -> CL10B104KA8NNNC
- C_U4_IN, C_U4_OUT: DK_PN (none) -> 1276-1935-1-ND; MPN (none) -> CL10B105KA8NNNC
- D1, D_FAN: DK_PN (none) -> 1N4148W-FDICT-ND; MPN (none) -> 1N4148W-7-F
- D_12V, D_USB: DK_PN (none) -> MBR0530T1GOSCT-ND; MPN (none) -> MBR0530T1G
- F1, F2: DK_PN (none) -> F1197-ND; MPN (none) -> ATM-7.5
- F3: DK_PN (none) -> F1185-ND; MPN (none) -> ATM-2
- FB1: DK_PN (none) -> 490-BLM18KG601TN1DCT-ND; MPN (none) -> BLM18KG601TN1D
- FH1, FH2, FH3: DK_PN (none) -> BK-6013-ND; MPN (none) -> BK-6013
- J_DISP_I2C, J_NFC: DK_PN (none) -> 455-2249-ND; MPN (none) -> B4B-XH-A
- J_DISP_SPI: DK_PN (none) -> 455-2253-ND; MPN (none) -> B8B-XH-A
- J_FAN: DK_PN (none) -> WM4202-ND; MPN (none) -> 22-28-4023
- J_FAN_SEL: DK_PN (none) -> S1011EC-03-ND; MPN (none) -> PEC03SAAN
- J_LED: DK_PN (none) -> 455-1577-1-ND; MPN (none) -> BM03B-GHS-TBT
- J_PWR_A: DK_PN (none) -> ED2942-ND; MPN (none) -> OSTYK42105030
- J_PWR_B: DK_PN (none) -> ED2940-ND; MPN (none) -> OSTYK42102030
- J_SW1, J_SW2, J_SW3: DK_PN (none) -> 455-1576-1-ND; MPN (none) -> BM02B-GHS-TBT
- J_SWD: DK_PN (none) -> 3220-10-0100-00-ND; MPN (none) -> 3220-10-0100-00
- J_USB: DK_PN (none) -> 2073-USB4085-GF-ACT-ND; MPN (none) -> USB4085-GF-A
- K1: DK_PN (none) -> Z682-ND; MPN (none) -> G5LE-14-DC3
- L1: DK_PN (none) -> SRR4028-3R9YCT-ND; MPN (none) -> SRR4028-3R9Y
- L2: DK_PN (none) -> SRR4028-4R7YCT-ND; MPN (none) -> SRR4028-4R7Y
- LED_DBG1, LED_DBG2: DK_PN (none) -> XL-5050RGBC-WS2812B-ND; MPN (none) -> XL-5050RGBC-WS2812B
- Q1: DK_PN (none) -> AO3401A-ND; MPN (none) -> AO3401A
- Q2, Q3_DRV: DK_PN (none) -> MMBT2222ALT1GOSCT-ND; MPN (none) -> MMBT2222ALT1G
- Q3: DK_PN (none) -> IRFZ44NPBF-ND; MPN (none) -> IRFZ44NPBF
- Q4: DK_PN (none) -> IRLML2502TRPBFCT-ND; MPN (none) -> IRLML2502TRPBF
- RT1: DK_PN (none) -> 445-2160-1-ND; MPN (none) -> NTCG063JF103FTB
- R_12V_H, R_BAT_H, R_CHG_H: DK_PN (none) -> 311-68.0KHRCT-ND; MPN (none) -> RC0603FR-0768KL
- R_12V_L, R_BAT_L, R_BOOT0, R_CHG_L, R_G1: DK_PN (none) -> 311-10.0KHRCT-ND; MPN (none) -> RC0603FR-0710KL
- R_B3, R_I2C1_SCL, R_I2C1_SDA: DK_PN (none) -> 311-4.70KHRCT-ND; MPN (none) -> RC0603FR-074K7L
- R_BLEED1, R_BLEED2: DK_PN (none) -> SQP500JB-10R-ND; MPN (none) -> SQP500JB-10R
- R_BOOT_G3, R_FAN_PD, R_PG: DK_PN (none) -> 311-100KHRCT-ND; MPN (none) -> RC0603FR-07100KL
- R_CC1, R_CC2: DK_PN (none) -> 311-5.10KHRCT-ND; MPN (none) -> RC0603FR-075K1L
- R_FAN_G, R_G3, R_NTC_S: DK_PN (none) -> 311-100HRCT-ND; MPN (none) -> RC0603FR-07100RL
- R_GATE_K1: DK_PN (none) -> 311-1.00KHRCT-ND; MPN (none) -> RC0603FR-071KL
- R_LED_DIN: DK_PN (none) -> 311-470HRCT-ND; MPN (none) -> RC0603FR-07470RL
- R_SHUNT: DK_PN (none) -> WSL2512R0100FEK18CT-ND; MPN (none) -> WSL2512R0100FEK18
- SW_BOOT, SW_RST: DK_PN (none) -> SW400-ND; MPN (none) -> B3F-4050
- U1: DK_PN (none) -> 497-STM32G0B1CCT6-ND; MPN (none) -> STM32G0B1CCT6
- U3: DK_PN (none) -> AP63203WU-7DICT-ND; MPN (none) -> AP63203WU-7
- U4: DK_PN (none) -> 576-1281-1-ND; MPN (none) -> MIC5219-3.3YM5-TR
- U5: DK_PN (none) -> AP63205WU-7DICT-ND; MPN (none) -> AP63205WU-7

Commit message: schematic wiring done
Co-Authored-By: Claude Opus 4.6 (1M context) <noreply@anthropic.com>
Parts:
- added U2: INA226AQDGSRQ1, INA226AQDGSRQ1:DGS10_TEX, symbol INA226AQDGSRQ1:INA226AQDGSRQ1

Commit message: fixed instance reference designators
Co-Authored-By: Claude Opus 4.6 (1M context) <noreply@anthropic.com>
Parts:
- removed D1: 1N4148W, Diode_SMD:D_SOD-123, symbol Device:D_Schottky
- removed F1, F2: 7.5A, Fuse:Fuse_Blade_ATM_Mini, symbol Device:Fuse
- removed F3: 2A, Fuse:Fuse_Blade_ATM_Mini, symbol Device:Fuse
- removed FH1, FH2, FH3: BK-6013, Fuse:Fuse_Blade_ATM_Mini, symbol Device:Fuse
- removed J_PWR_A: OSTYK42105030, TerminalBlock_OnShore:TerminalBlock_OnShore_OSTTE050161_1x05_P5.08mm_Horizontal, symbol Connector:Screw_Terminal_01x05
- removed J_PWR_B: OSTYK42102030, TerminalBlock_OnShore:TerminalBlock_OnShore_OSTTE020161_1x02_P5.08mm_Horizontal, symbol Connector:Screw_Terminal_01x02
- removed K1: G5LE-1, Relay_THT:Relay_SPDT_Omron-G5LE-1, symbol Relay:G5LE-1
- removed Q1: AO3401A, Package_TO_SOT_SMD:SOT-23, symbol Transistor_FET:AO3401A
- removed Q2, Q3_DRV: MMBT2222A, Package_TO_SOT_SMD:SOT-23, symbol Transistor_BJT:MMBT2222A
- removed Q3: IRFZ44NPBF, Package_TO_SOT_THT:TO-220-3_Vertical, symbol Transistor_FET:IRLZ44N
- removed R_B3: 4k7, Resistor_SMD:R_0603_1608Metric, symbol Device:R
- removed R_BLEED1, R_BLEED2: 10R 5W, Resistor_THT:R_Axial_DIN0516_L15.5mm_D5.3mm_P22.86mm_Horizontal, symbol Device:R
- removed R_BOOT_G3: 100k, Resistor_SMD:R_0603_1608Metric, symbol Device:R
- removed R_G1: 10k, Resistor_SMD:R_0603_1608Metric, symbol Device:R
- removed R_G3: 100R, Resistor_SMD:R_0603_1608Metric, symbol Device:R
- removed R_GATE_K1: 1k, Resistor_SMD:R_0603_1608Metric, symbol Device:R
- removed R_SHUNT: 10m, Resistor_SMD:R_2512_6332Metric, symbol Device:R_Shunt
- renumbered C_12V_IN to C_12V_IN1, C_5V_IN to C_5V_IN1, C_5V_OUT to C_5V_OUT1, C_BST to C_BST1, C_BULK_3V3 to C_BULK_3V1, C_IN to C_IN1, C_INA_VS to C_INA_VS1, C_NRST to C_NRST1, C_OUT to C_OUT1, C_U4_IN to C_U4_IN1, C_U4_OUT to C_U4_OUT1, C_VBAT to C_VBAT1, C_VDDIO2 to C_VDDIO1, C_VDD_BULK to C_VDD_BULK1, C_VREF to C_VREF1, D_12V to D_12V1, D_FAN to D_FAN1, D_USB to D_USB1, J_DISP_I2C to J_DISP_I2C1, J_DISP_SPI to J_DISP_SPI1, J_EXP_A to J_EXP_A1, J_EXP_B to J_EXP_B1, J_FAN to J_FAN1, J_FAN_SEL to J_FAN_SEL1, J_LED to J_LED1, J_NFC to J_NFC1, J_SWD to J_SWD1, J_UART to J_UART1, J_USB to J_USB1, R_12V_H to R_12V_H1, R_12V_L to R_12V_L1, R_BAT_H to R_BAT_H1, R_BAT_L to R_BAT_L1, R_BOOT0 to R_BOOT1, R_CHG_H to R_CHG_H1, R_CHG_L to R_CHG_L1, R_FAN_G to R_FAN_G1, R_FAN_PD to R_FAN_PD1, R_I2C1_SCL to R_I2C1_SCL1, R_I2C1_SDA to R_I2C1_SDA1, R_LED_DIN to R_LED_DIN1, R_NTC_S to R_NTC_S1, R_PG to R_PG1, SW_BOOT to SW_BOOT1, SW_RST to SW_RST1
