File: 1-BatteryPowerPath.kicad_sch (KiCad schematic)
At the start: 0 parts

Commit message: fixed instance reference designators
Co-Authored-By: Claude Opus 4.6 (1M context) <noreply@anthropic.com>
Parts:
- added D1: 1N4148W, Diode_SMD:D_SOD-123, symbol Device:D_Schottky
- added F1, F2: 7.5A, Fuse:Fuse_Blade_ATM_Mini, symbol Device:Fuse
- added F3: 2A, Fuse:Fuse_Blade_ATM_Mini, symbol Device:Fuse
- added FH1, FH2, FH3: BK-6013, Fuse:Fuse_Blade_ATM_Mini, symbol Device:Fuse
- added J_PWR_A1: OSTYK42105030, TerminalBlock_OnShore:TerminalBlock_OnShore_OSTTE050161_1x05_P5.08mm_Horizontal, symbol Connector:Screw_Terminal_01x05
- added J_PWR_B1: OSTYK42102030, TerminalBlock_OnShore:TerminalBlock_OnShore_OSTTE020161_1x02_P5.08mm_Horizontal, symbol Connector:Screw_Terminal_01x02
- added K1: G5LE-1, Relay_THT:Relay_SPDT_Omron-G5LE-1, symbol Relay:G5LE-1
- added Q1: AO3401A, Package_TO_SOT_SMD:SOT-23, symbol Transistor_FET:AO3401A
- added Q2, Q3_DRV1: MMBT2222A, Package_TO_SOT_SMD:SOT-23, symbol Transistor_BJT:MMBT2222A
- added Q3: IRFZ44NPBF, Package_TO_SOT_THT:TO-220-3_Vertical, symbol Transistor_FET:IRLZ44N
- added R_B1: 4k7, Resistor_SMD:R_0603_1608Metric, symbol Device:R
- added R_BLEED1, R_BLEED2: 10R 5W, Resistor_THT:R_Axial_DIN0516_L15.5mm_D5.3mm_P22.86mm_Horizontal, symbol Device:R
- added R_BOOT_G1: 100k, Resistor_SMD:R_0603_1608Metric, symbol Device:R
- added R_G1: 10k, Resistor_SMD:R_0603_1608Metric, symbol Device:R
- added R_G2: 100R, Resistor_SMD:R_0603_1608Metric, symbol Device:R
- added R_GATE_K1: 1k, Resistor_SMD:R_0603_1608Metric, symbol Device:R
- added R_SHUNT1: 10m, Resistor_SMD:R_2512_6332Metric, symbol Device:R_Shunt
