File: BatteryMonitorModule/02-PowerSupply.kicad_sch (KiCad schematic)
At the start: 0 parts

Commit message: schematic annotation and component placement for power supply, MCU, and power path sheets
Added symbol libraries (AP63203, AP63205, MIC5219, TC2117), annotated
ref designators, and placed components via MCP server. Includes
fix_sheet_instances.py utility for restoring sheet_instances blocks.

Co-Authored-By: Claude Opus 4.6 (1M context) <noreply@anthropic.com>
Parts:
- added C1, C4, C5: 10uF, symbol Device:C
- added C2: 22uF, symbol Device:C
- added C3: 100nF, symbol Device:C
- added D2: MBR0530, symbol Device:D_Schottky
- added FH3: 2A ATM, symbol Device:Fuse
- added J2: OSTYK42102030, symbol Connector:Screw_Terminal_01x02
- added L1: 4.7uH, symbol Device:L
- added R25: 33k, symbol Device:R
- added R26: 82k, symbol Device:R
- added U3: AP63205WU-7, symbol AP63205WU-7:AP63205WU-7
- added U4: TC2117-3.3VDBTR, symbol TC2117-3.3VDBTR:TC2117-3.3VDBTR
Connections:
- new net: C3.2, L1.1, U3.5 (SW)
- new net: FH3.1, J2.1 (Pin_1)
- new net: C3.1, U3.6 (BST)
- new net +12V: C1.1, C4.2, FH3.2, U3.3 (VIN)
- new net +3.3V: C5.1, U4.3 (OUT)
- new net +5V: C2.1, D2.1 (K), L1.2, U3.1 (FB), U3.2 (EN), U4.1 (IN)
- new net +5VUsb: D2.2 (A), R25.2
- new net GND: C1.2, C2.2, C4.1, C5.2, J2.2 (Pin_2), R26.1, U3.4 (GND), U4.2 (GND)
- new net VBUS_SENSE: R25.1, R26.2
Other:
- note added: "12->5V"
- note added: "5V USB Bus -> Diode ->5V bus Nominally USB at 5.25 or lower won't pass unless no 12 V present. 12V -> 5V Regulator is pulled up to always enable in either 12 or usb connected This means if no 12V present enters LV protection Does not pull 5V low so 5VUSB will dominate."
- note added: "5V->3.3 LDO"

Commit message: updated power supply schematic — additional component placement and wiring
Co-Authored-By: Claude Opus 4.6 (1M context) <noreply@anthropic.com>
Changed lines of the file:
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@@
+	)
+	(junction
+		(at 147.32 36.83)
+		(diameter 0)
+		(color 0 0 0 0)
 	)
 	(junction
@@
 	)
 	(symbol
+		(lib_id "power:PWR_FLAG")
+		(at 44.45 49.53 180)
+		(unit 1)
+		(exclude_from_sim no)
+		(in_bom yes)
+		(on_board yes)
+		(dnp no)
+		(fields_autoplaced yes)
+		(property "Reference" "#FLG01"
+			(at 44.45 51.435 0)
+			(effects
+				(font
+					(size 1.27 1.27)
+				)
+				(hide yes)
+			)
+		)
+		(property "Value" "PWR_FLAG"
+			(at 44.45 54.61 0)
+			(effects
+				(font
+					(size 1.27 1.27)
+				)
+			)
+		)
+		(property "Footprint" ""
+			(at 44.45 49.53 0)
+			(effects
+				(font
+					(size 1.27 1.27)
+				)
+				(hide yes)
+			)
+		)
+		(property "Datasheet" "~"
+			(at 44.45 49.53 0)
+			(effects
+				(font
+					(size 1.27 1.27)
+				)
+				(hide yes)
+			)
+		)
+		(property "Description" "Special symbol for telling ERC where power comes from"
+			(at 44.45 49.53 0)
+			(effects
+				(font
+					(size 1.27 1.27)
+				)
+				(hide yes)
+			)
+		)
+		(pin "1"
+		)
+		(instances
+			(project "BatteryMonitorModule"
+				(path "/03269402-9c05-492f-98b8-b4c760268d66/b2000002-0000-0000-0000-000000000002"
+					(reference "#FLG01")
+					(unit 1)
+				)
+			)
+		)
+	)
+	(symbol
 		(lib_id "TC2117-3.3VDBTR:TC2117-3.3VDBTR")
 		(at 95.25 87.63 0)
@@
 					(unit 1)
 				)
+			)
+		)
+	)
+	(symbol
+		(lib_id "power:PWR_FLAG")
+		(at 147.32 36.83 0)
+		(unit 1)
+		(exclude_from_sim no)
+		(in_bom yes)
+		(on_board yes)
+		(dnp no)
+		(fields_autoplaced yes)
+		(property "Reference" "#FLG02"
+			(at 147.32 34.925 0)
+			(effects
+				(font
+					(size 1.27 1.27)
+				)
+				(hide yes)
+			)
+		)
+		(property "Value" "PWR_FLAG"
+			(at 147.32 31.75 0)
+			(effects
+				(font
+					(size 1.27 1.27)
+				)
+			)
+		)
+		(property "Footprint" ""
+			(at 147.32 36.83 0)
+			(effects
+				(font
+					(size 1.27 1.27)
+				)
+				(hide yes)
+			)
+		)
+		(property "Datasheet" "~"
+			(at 147.32 36.83 0)
+			(effects
+				(font
+					(size 1.27 1.27)
+				)
+				(hide yes)
+			)
+		)
+		(property "Description" "Special symbol for telling ERC where power comes from"
+			(at 147.32 36.83 0)
+			(effects
+				(font
+					(size 1.27 1.27)
+				)
+				(hide yes)
+			)
+		)
+		(pin "1"
+		)
+		(instances
+			(project "BatteryMonitorModule"
+				(path "/03269402-9c05-492f-98b8-b4c760268d66/b2000002-0000-0000-0000-000000000002"
+					(reference "#FLG02")
+					(unit 1)
+				)

Commit message: updated all schematics — IO sheet wiring, MCU connections, power supply refinements, custom footprints
Co-Authored-By: Claude Opus 4.6 (1M context) <noreply@anthropic.com>
Parts:
- C1, C2, C4, C5: footprint (none) -> Capacitor_SMD:C_0805_2012Metric
- C3: footprint (none) -> Capacitor_SMD:C_0603_1608Metric
- D2: footprint (none) -> Diode_SMD:D_SOD-123
- FH3: footprint (none) -> Fuse:FuseHolder_Blade_ATO_Littelfuse_FLR_178.6165
- J2: footprint (none) -> TerminalBlock_Phoenix:TerminalBlock_Phoenix_MKDS-1,5-2-5.08_1x02_P5.08mm_Horizontal
- L1: footprint (none) -> BatteryMonitorModule_Custom:IND_BOURNS_SRR4028
- R25, R26: footprint (none) -> Resistor_SMD:R_0603_1608Metric
- U3: footprint (none) -> BatteryMonitorModule_Custom:AP63205WU-7_DIO
- U4: footprint (none) -> Package_TO_SOT_SMD:SOT-223-3_TabPin2

Commit message: added connector footprints and power path updates
New custom footprints: OSTYK screw terminals, KF8500 connectors, USB4085-GF-A.
Power path schematic updates and project library references.

Co-Authored-By: Claude Opus 4.6 (1M context) <noreply@anthropic.com>
Parts:
- J2: footprint TerminalBlock_Phoenix:TerminalBlock_Phoenix_MKDS-1,5-2-5.08_1x02_P5.08mm_Horizontal -> BatteryMonitorModule_Custom:OSTYK42102030
Changed lines of the file:
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@@
 			)
 		)
-		(property "Footprint" "TerminalBlock_Phoenix:TerminalBlock_Phoenix_MKDS-1,5-2-5.08_1x02_P5.08mm_Horizontal"
+		(property "Footprint" "BatteryMonitorModule_Custom:OSTYK42102030"
 			(at 25.4 49.53 0)
 			(hide yes)
