File: BatteryMonitorModule/02-PowerSupply.kicad_sch (KiCad schematic)
At the start: 14 parts, among them J2 OSTYK42102030, U3 AP63205WU-7, U4 TC2117-3.3VDBTR

Commit message: added 3D models, updated footprints, and schematic/PCB updates
New 3D STEP models: AP63205, BK-6013 fuse holder, FSMSM switch,
SRR4028 inductor, OSTYK screw terminals, USB4085, WSK2512 shunt,
SQP500 resistor. Updated custom footprints with 3D model references.
New BK-6013 fuse holder footprint.

Co-Authored-By: Claude Opus 4.6 (1M context) <noreply@anthropic.com>
Parts:
- C1, C2, C3, C5, R25, R26: KiLib_Generator (none) -> SMD_2terminal_chip_molded
- FH3: footprint Fuse:FuseHolder_Blade_ATO_Littelfuse_FLR_178.6165 -> BatteryMonitorModule_Custom:FUSE_BK-6013
Changed lines of the file:
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@@
+			)
+		)
+		(property "KiLib_Generator" "SMD_2terminal_chip_molded"
+			(at 39.37 76.2 0)
+			(hide yes)
+			(show_name no)
+			(do_not_autoplace no)
+			(effects
+				(font
+					(size 1.27 1.27)
+				)
 			)
 		)
@@
 		(property "Description" ""
 			(at 118.11 97.79 0)
+			(show_name no)
+			(do_not_autoplace no)
+			(effects
+				(font
+					(size 1.27 1.27)
+				)
+			)
+		)
+		(property "KiLib_Generator" "SMD_2terminal_chip_molded"
+			(at 118.11 97.79 0)
+			(hide yes)
 			(show_name no)
 			(do_not_autoplace no)
@@
 			)
 		)
+		(property "KiLib_Generator" "SMD_2terminal_chip_molded"
+			(at 77.47 58.42 0)
+			(hide yes)
+			(show_name no)
+			(do_not_autoplace no)
+			(effects
+				(font
+					(size 1.27 1.27)
+				)
+			)
+		)
 		(pin "1"
 		)
@@
 			)
 		)
-		(property "Footprint" "Fuse:FuseHolder_Blade_ATO_Littelfuse_FLR_178.6165"
+		(property "Footprint" "BatteryMonitorModule_Custom:FUSE_BK-6013"
 			(at 38.1 49.53 0)
 			(hide yes)
@@
 			)
 		)
+		(property "KiLib_Generator" "SMD_2terminal_chip_molded"
+			(at 39.37 87.63 0)
+			(hide yes)
+			(show_name no)
+			(do_not_autoplace no)
+			(effects
+				(font
+					(size 1.27 1.27)
+				)
+			)
+		)
 		(pin "1"
 		)
@@
 		(property "Description" ""
 			(at 147.32 55.88 0)
+			(show_name no)
+			(do_not_autoplace no)
+			(effects
+				(font
+					(size 1.27 1.27)
+				)
+			)
+		)
+		(property "KiLib_Generator" "SMD_2terminal_chip_molded"
+			(at 147.32 55.88 0)
+			(hide yes)
 			(show_name no)
 			(do_not_autoplace no)
@@
 			(show_name no)
 			(do_not_autoplace no)
+			(effects
+				(font
+					(size 1.27 1.27)
+				)
+			)
+		)
+		(property "KiLib_Generator" "SMD_2terminal_chip_molded"
+			(at 129.54 46.99 0)
+			(hide yes)
+			(show_name no)
+			(do_not_autoplace no)

Commit message: V0 design updates — PCB layout refinements and power supply schematic fixes
Co-Authored-By: Claude Opus 4.6 <noreply@anthropic.com>
Parts:
- R25: value 33k -> 82k
- R26: value 82k -> 33k
Changed lines of the file:
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@@
 			)
 		)
-		(property "Value" "33k"
+		(property "Value" "82k"
 			(at 39.116 76.2 90)
 			(show_name no)
@@
 			)
 		)
-		(property "Value" "82k"
+		(property "Value" "33k"
 			(at 39.464 87.63 90)
 			(show_name no)
