File: BatteryMonitorModule/03-MCU.kicad_sch (KiCad schematic)
At the start: 19 parts, among them J3 Conn_ARM_JTAG_SWD_10, J4 USB-C, SW1 BOOT0, SW2 NRST, U1 STM32G0B1CCT6, U2 INA226AQDGSRQ1

Commit message: routed
Parts:
- removed C9: 100nF, Capacitor_SMD:C_0603_1608Metric, symbol Device:C
- removed FB1: 600R@100MHz, Inductor_SMD:L_0603_1608Metric, symbol Device:L
Connections:
- net GND: now also U2.7 (GND)
