File: BatteryMonitorModule/04-IO.kicad_sch (KiCad schematic)
At the start: 29 parts, among them J10 J_DISP_SPI, J11 J_UART, J12 J_EXP_B, J13 J_EXP_A, J5 J_FAN, J6 J_FAN_SEL, J7 J_NFC, J8 J_PANEL, Q5 2N7002

Commit message: added 3D models, updated footprints, and schematic/PCB updates
New 3D STEP models: AP63205, BK-6013 fuse holder, FSMSM switch,
SRR4028 inductor, OSTYK screw terminals, USB4085, WSK2512 shunt,
SQP500 resistor. Updated custom footprints with 3D model references.
New BK-6013 fuse holder footprint.

Co-Authored-By: Claude Opus 4.6 (1M context) <noreply@anthropic.com>
Parts:
- J10, J7, J8: KiLib_Generator (none) -> connector/JST
- J11, J12, J13, J5, J6: KiLib_Generator (none) -> connector/pin_header_socket
- LED3, LED4, LED5, LED6, R16, R17, R18, R19, R20, R21, R22, R23, R24, R29, R30, R31, R34: KiLib_Generator (none) -> SMD_2terminal_chip_molded
- Q5: KiLib_Generator (none) -> package/gullwing
