File: BatteryMonitorModule/BatteryMonitorModule.kicad_pcb (KiCad board)
At the start: 2 copper layers, 76.2 x 101.6 mm, 85 parts, among them J1 OSTYK42105030, J10 J_DISP_SPI, J11 J_UART, J12 J_EXP_B, J13 J_EXP_A, J2 OSTYK42102030, J3 Conn_ARM_JTAG_SWD_10, J4 USB-C, J5 J_FAN, J6 J_FAN_SEL, J7 J_NFC, J8 J_PANEL, K1 G5LE-1, Q1 AO3401A, Q2 IRFZ44NPBF, Q3 MMBT2222A, Q4 MMBT2222A, Q5 2N7002, SW1 BOOT0, SW2 NRST, U1 STM32G0B1CCT6, U2 INA226AQDGSRQ1, U3 AP63205WU-7, U4 TC2117-3.3VDBTR

Commit message: added 3D models, updated footprints, and schematic/PCB updates
New 3D STEP models: AP63205, BK-6013 fuse holder, FSMSM switch,
SRR4028 inductor, OSTYK screw terminals, USB4085, WSK2512 shunt,
SQP500 resistor. Updated custom footprints with 3D model references.
New BK-6013 fuse holder footprint.

Co-Authored-By: Claude Opus 4.6 (1M context) <noreply@anthropic.com>
Parts:
- F1, F2, FH3: footprint Fuse:FuseHolder_Blade_ATO_Littelfuse_FLR_178.6165 -> BatteryMonitorModule_Custom:FUSE_BK-6013
- moved J8 12.8 mm to (81.2, 123.0), turned to 180 degrees
- moved J7 8.02 mm to (97.5, 51.5), turned to -90 degrees
- moved FH3 5.14 mm to (75.8, 43.5)
- moved F2 4.46 mm to (64.5, 48.4)
- moved F1 3.50 mm to (37.0, 48.0)
Routing:
- net Net-(J1-Pin_1): track 29.9 -> 9.47 mm
- net +3.3V: track 230.2 -> 211.2 mm
- net Net-(J2-Pin_1): track 20.4 -> 6.93 mm
- net Net-(J1-Pin_3): track 29.0 -> 16.4 mm
- net SW_A: track 55.6 -> 65.0 mm
- net /04-IO/LED_DATA_O: track 17.8 -> 8.63 mm
- net Net-(F1-Pad2): track 21.4 -> 12.7 mm
- net +5V: track 154.8 -> 148.1 mm, vias 1 -> 0
- net I2C1_SCL: track 105.1 -> 110.6 mm, vias 6 -> 5
- net GND: track 189.3 -> 184.9 mm, vias 34 -> 33
- net CHG_P_F2: track 35.8 -> 38.3 mm
- net SW_C: track 57.1 -> 59.3 mm
- net USB_DP: track 82.5 -> 84.7 mm
- net USB_DN: track 84.8 -> 86.8 mm
- net SW_B: track 56.8 -> 54.8 mm
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