File: BatteryMonitorModule/BatteryMonitorModule.kicad_pcb (KiCad board)
At the start: 2 copper layers, 76.2 x 101.6 mm, 85 parts, among them J1 OSTYK42105030, J10 J_DISP_SPI, J11 J_UART, J12 J_EXP_B, J13 J_EXP_A, J2 OSTYK42102030, J3 Conn_ARM_JTAG_SWD_10, J4 USB-C, J5 J_FAN, J6 J_FAN_SEL, J7 J_NFC, J8 J_PANEL, K1 G5LE-1, Q1 AO3401A, Q2 IRFZ44NPBF, Q3 MMBT2222A, Q4 MMBT2222A, Q5 2N7002, SW1 BOOT0, SW2 NRST, U1 STM32G0B1CCT6, U2 INA226AQDGSRQ1, U3 AP63205WU-7, U4 TC2117-3.3VDBTR

Commit message: design done commit
Parts:
- removed REF** (x4): MountingHole_3.2mm_M3, MountingHole:MountingHole_3.2mm_M3
- added H1: MountingHole_Pad, MountingHole:MountingHole_3.2mm_M3_DIN965_Pad, F.Cu at (98.0, 29.0)
- added H2: MountingHole_Pad, MountingHole:MountingHole_3.2mm_M3_DIN965_Pad, F.Cu at (29.0, 29.0)
- added H3: MountingHole_Pad, MountingHole:MountingHole_3.2mm_M3_DIN965_Pad, F.Cu at (29.0, 123.5)
- added H4: MountingHole_Pad, MountingHole:MountingHole_3.2mm_M3_DIN965_Pad, F.Cu at (98.0, 123.5)
- J4: footprint BatteryMonitorModule_Custom:USB4085-GF-A_GCT -> BatteryMonitorModule_Custom:GCT_USB4085-GF-A_REVA4
- U2: footprint Package_SO:MSOP-10_3x3mm_P0.5mm -> Package_SO:TSSOP-10_3x3mm_P0.5mm
- moved R12 31.6 mm to (49.0, 91.0), turned to 0 degrees
- moved R11 28.0 mm to (49.0, 89.0), turned to 0 degrees
- moved J4 5.15 mm to (99.0, 41.6)
- moved Q3 4.44 mm to (41.1, 92.0)
- moved R4 4.20 mm to (44.0, 94.6)
- moved R14 4.12 mm to (98.1, 34.6)
- moved R5 3.95 mm to (45.0, 92.0)
- moved C10 0.89 mm to (54.0, 56.0)
- moved R15 0.78 mm to (96.5, 34.6)
Connections:
- R14 pad 1: Net-(J4-CC1) -> Net-(J4-CC2)
- R15 pad 1: Net-(J4-CC2) -> Net-(J4-CC1)
Routing:
- net GND: track 184.9 -> 317.7 mm, vias 33 -> 48
- net +3.3V: track 211.2 -> 289.5 mm
- net VBUS_SENSE: track 1.86 -> 54.2 mm, vias 0 -> 4
- net ADC_12V: track 0.00 -> 48.4 mm, vias 0 -> 2
- net /04-IO/LED_DATA_O: track 8.63 -> 32.5 mm
- net J13-5: track 70.6 -> 49.9 mm, vias 0 -> 2
- net SW_C: track 59.3 -> 54.2 mm, vias 0 -> 1
- net GPIO_BLEED: track 30.3 -> 34.4 mm, vias 2 -> 4
- net Net-(J2-Pin_1): track 6.93 -> 10.6 mm
- net +12V: track 170.9 -> 174.6 mm, vias 5 -> 4
- net CHG_P_F2: track 38.3 -> 41.7 mm, vias 0 -> 1
- net Net-(Q3-C): track 2.69 -> 5.34 mm
- net I2C1_SCL: track 110.6 -> 108.4 mm, vias 5 -> 6
- net USB_DN: track 86.8 -> 85.0 mm
- net I2C1_SDA: track 110.2 -> 108.5 mm, vias 5 -> 6
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