File: BatteryMonitorModule/BatteryMonitorModule.kicad_pcb (KiCad board)
At the start: 2 copper layers, 76.2 x 101.6 mm, 85 parts, among them J1 OSTYK42105030, J10 J_DISP_SPI, J11 J_UART, J12 J_EXP_B, J13 J_EXP_A, J2 OSTYK42102030, J3 Conn_ARM_JTAG_SWD_10, J4 USB-C, J5 J_FAN, J6 J_FAN_SEL, J7 J_NFC, J8 J_PANEL, K1 G5LE-1, Q1 AO3401A, Q2 IRFZ44NPBF, Q3 MMBT2222A, Q4 MMBT2222A, Q5 2N7002, SW1 BOOT0, SW2 NRST, U1 STM32G0B1CCT6, U2 INA226AQDGSRQ1, U3 AP63205WU-7, U4 TC2117-3.3VDBTR

Commit message: V0 design updates — PCB layout refinements and power supply schematic fixes
Co-Authored-By: Claude Opus 4.6 <noreply@anthropic.com>
Parts:
- R25: value 33k -> 82k
- R26: value 82k -> 33k
- U2: footprint Package_SO:TSSOP-10_3x3mm_P0.5mm -> Package_SO:MSOP-10_3x3mm_P0.5mm
Other:
- board text added: "www.github.com/tuffinmuffin Rev - Battery Monitoring Module"
Changed lines of the file:
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@@
 		(capping no)
 		(filling no)
-		(zone_defaults)
 		(pcbplotparams
 			(layerselection 0x00000000_00000000_55555555_5755f5ff)
@@
 			(outputformat 1)
 			(mirror no)
-			(drillshape 1)
+			(drillshape 0)
 			(scaleselection 1)
-			(outputdirectory "")
+			(outputdirectory "BatteryMonitor-Rev-/")
 		)
 	)
@@
 		(sheetname "/02-PowerSupply/")
 		(sheetfile "02-PowerSupply.kicad_sch")
+		(units
+			(unit
+				(name "A")
+				(pins "1" "2")
+			)
+		)
 		(attr through_hole)
 		(duplicate_pad_numbers_are_jumpers no)
@@
 			)
 		)
-		(property "Value" "82k"
+		(property "Value" "33k"
 			(at 0 1.43 90)
 			(layer "F.Fab")
@@
 		(sheetname "/02-PowerSupply/")
 		(sheetfile "02-PowerSupply.kicad_sch")
+		(units
+			(unit
+				(name "A")
+				(pins "1" "2")
+			)
+		)
 		(attr smd)
 		(duplicate_pad_numbers_are_jumpers no)
@@
 			)
 		)
-		(property "Value" "33k"
+		(property "Value" "82k"
 			(at 0 1.43 90)
 			(layer "F.Fab")
@@
 		)
 	)
-	(footprint "Package_SO:TSSOP-10_3x3mm_P0.5mm"
+	(footprint "Package_SO:MSOP-10_3x3mm_P0.5mm"
 		(layer "F.Cu")
 		(at 56.1 60 180)
-		(descr "TSSOP, 10 Pin (https://www.ti.com/lit/ml/mpds035c/mpds035c.pdf, https://www.ti.com/lit/ds/symlink/ads1115.pdf#page=50, https://www.nxp.com/docs/en/package-information/SOT552-1.pdf)")
-		(tags "TSSOP SO Texas_DGS0010A Texas_VSSOP-10 NXP_SOT552-1 MSOP-10_3x3mm_P0.5mm VSSOP-10_3x3mm_P0.5mm")
+		(descr "MSOP, 10 Pin (JEDEC MO-187 variation BA, 0.85mm body thickness, https://www.jedec.org/system/files/docs/mo-187F.pdf)")
+		(tags "MSOP SO TSSOP-10_3x3mm_P0.5mm")
 		(property "Reference" "U2"
-			(at 2.1 -2.45 180)
+			(at 0 -2.45 180)
 			(layer "F.SilkS")
 			(effects
@@
 		(sheetname "/03-MCU/")
 		(sheetfile "03-MCU.kicad_sch")
+		(units
+			(unit
+				(name "A")
+				(pins "1" "2" "3" "4" "5" "10" "9" "8" "7" "6")
+			)
+		)
 		(attr smd)
 		(duplicate_pad_numbers_are_jumpers no)
@@
 		)
 		(fp_line
-			(start 1.61 1.41)
+			(start 1.61 1.435)
 			(end 1.61 1.61)
 			(stroke
@@
 		(fp_line
 			(start 1.61 -1.61)
-			(end 1.61 -1.41)
+			(end 1.61 -1.435)
 			(stroke
 				(width 0.12)
@@
 		(fp_line
 			(start -1.61 1.61)
-			(end -1.61 1.41)
+			(end -1.61 1.435)
 			(stroke
 				(width 0.12)
@@
 		)
 		(fp_line
-			(start -1.61 -1.41)
+			(start -1.61 -1.435)
 			(end -1.61 -1.61)
 			(stroke
@@
 		(fp_poly
 			(pts
-				(xy -2.16 -1.41) (xy -2.4 -1.74) (xy -1.92 -1.74)
+				(xy -2.16 -1.44) (xy -2.4 -1.77) (xy -1.92 -1.77)
 			)
 			(stroke
@@
 		)
 		(fp_line
-			(start 3.13 1.4)
-			(end 1.75 1.4)
+			(start 3.1 1.43)
+			(end 1.75 1.43)
 			(stroke
 				(width 0.05)
@@
 		)
 		(fp_line
-			(start 3.13 -1.4)
-			(end 3.13 1.4)
+			(start 3.1 -1.43)
+			(end 3.1 1.43)
 			(stroke
 				(width 0.05)
@@
 		)
 		(fp_line
-			(start 1.75 1.4)
+			(start 1.75 1.43)
 			(end 1.75 1.75)
 			(stroke
@@
 		)
 		(fp_line
-			(start 1.75 -1.4)
-			(end 3.13 -1.4)
+			(start 1.75 -1.43)
+			(end 3.1 -1.43)
 			(stroke
 				(width 0.05)
@@
 		(fp_line
 			(start 1.75 -1.75)
-			(end 1.75 -1.4)
+			(end 1.75 -1.43)
 			(stroke
 				(width 0.05)
@@
 		(fp_line
 			(start -1.75 1.75)
-			(end -1.75 1.4)
+			(end -1.75 1.43)
 			(stroke
 				(width 0.05)
@@
 		)
 		(fp_line
-			(start -1.75 1.4)
-			(end -3.13 1.4)
+			(start -1.75 1.43)
+			(end -3.1 1.43)
 			(stroke
 				(width 0.05)
@@
 		)
 		(fp_line
-			(start -1.75 -1.4)
+			(start -1.75 -1.43)
 			(end -1.75 -1.75)
 			(stroke
@@
 		)
 		(fp_line
-			(start -3.13 1.4)
-			(end -3.13 -1.4)
+			(start -3.1 1.43)
+			(end -3.1 -1.43)
 			(stroke
 				(width 0.05)
@@
 		)
 		(fp_line
-			(start -3.13 -1.4)
-			(end -1.75 -1.4)
+			(start -3.1 -1.43)
+			(end -1.75 -1.43)
 			(stroke
 				(width 0.05)
@@
 		)
 		(pad "1" smd roundrect
-			(at -2.15 -1 180)
-			(size 1.45 0.3)
+			(at -2.1 -1 180)
+			(size 1.5 0.35)
 			(layers "F.Cu" "F.Mask" "F.Paste")
 			(roundrect_rratio 0.25)
@@
 		)
 		(pad "2" smd roundrect
-			(at -2.15 -0.5 180)
-			(size 1.45 0.3)
+			(at -2.1 -0.5 180)
+			(size 1.5 0.35)
 			(layers "F.Cu" "F.Mask" "F.Paste")
 			(roundrect_rratio 0.25)
@@
 		)
 		(pad "3" smd roundrect
-			(at -2.15 0 180)
-			(size 1.45 0.3)
+			(at -2.1 0 180)
+			(size 1.5 0.35)
 			(layers "F.Cu" "F.Mask" "F.Paste")
 			(roundrect_rratio 0.25)
@@
 		)
 		(pad "4" smd roundrect
-			(at -2.15 0.5 180)
-			(size 1.45 0.3)
+			(at -2.1 0.5 180)
+			(size 1.5 0.35)
 			(layers "F.Cu" "F.Mask" "F.Paste")
 			(roundrect_rratio 0.25)
@@
 		)
 		(pad "5" smd roundrect
-			(at -2.15 1 180)
-			(size 1.45 0.3)
+			(at -2.1 1 180)
+			(size 1.5 0.35)
 			(layers "F.Cu" "F.Mask" "F.Paste")
 			(roundrect_rratio 0.25)
@@
 		)
 		(pad "6" smd roundrect
-			(at 2.15 1 180)
-			(size 1.45 0.3)
+			(at 2.1 1 180)
+			(size 1.5 0.35)
 			(layers "F.Cu" "F.Mask" "F.Paste")
 			(roundrect_rratio 0.25)
@@
 		)
 		(pad "7" smd roundrect
-			(at 2.15 0.5 180)
-			(size 1.45 0.3)
+			(at 2.1 0.5 180)
+			(size 1.5 0.35)
 			(layers "F.Cu" "F.Mask" "F.Paste")
 			(roundrect_rratio 0.25)
@@
 		)
 		(pad "8" smd roundrect
-			(at 2.15 0 180)
-			(size 1.45 0.3)
+			(at 2.1 0 180)
+			(size 1.5 0.35)
 			(layers "F.Cu" "F.Mask" "F.Paste")
 			(roundrect_rratio 0.25)
@@
 		)
 		(pad "9" smd roundrect
-			(at 2.15 -0.5 180)
-			(size 1.45 0.3)
+			(at 2.1 -0.5 180)
+			(size 1.5 0.35)
 			(layers "F.Cu" "F.Mask" "F.Paste")
 			(roundrect_rratio 0.25)
@@
 		)
 		(pad "10" smd roundrect
-			(at 2.15 -1 180)
-			(size 1.45 0.3)
+			(at 2.1 -1 180)
+			(size 1.5 0.35)
 			(layers "F.Cu" "F.Mask" "F.Paste")
 			(roundrect_rratio 0.25)
@@
 		)
 		(embedded_fonts no)
-		(model "${KICAD10_3DMODEL_DIR}/Package_SO.3dshapes/TSSOP-10_3x3mm_P0.5mm.step"
+		(model "${KICAD10_3DMODEL_DIR}/Package_SO.3dshapes/MSOP-10_3x3mm_P0.5mm.step"
 			(offset
 				(xyz 0 0 0)
@@
 		(sheetname "/03-MCU/")
 		(sheetfile "03-MCU.kicad_sch")
+		(units
+			(unit
+				(name "A")
+				(pins "A4" "A9" "B4" "B9" "A5" "B5" "A6" "B6" "A7" "B7" "A8" "B8" "S1"
+					"S2" "S3" "S4" "A1" "A12" "B1" "B12"
+				)
+			)
+		)
 		(attr through_hole)
 		(duplicate_pad_numbers_are_jumpers no)
@@
 		(layer "User.4")
 	)
+	(gr_text "www.github.com/tuffinmuffin\nRev -\nBattery\nMonitoring Module"
+		(at 84.5 123.5 0)
+		(layer "F.SilkS")
+		(effects
+			(font
+				(size 0.74 0.75)
+				(thickness 0.185)
+				(bold yes)
+			)
+			(justify left bottom)
+		)
+	)
 	(gr_text "+5V"
