File: CAD/BatteryMonitorModule_V1/BatteryMonitorModule/02-PowerSupply.kicad_sch (KiCad schematic)
At the start: 14 parts, among them J2 OSTYK42102030, U3 AP63205WU-7, U4 TC2117-3.3VDBTR

Commit message: V1 schematic rework — PowerPath, PowerSupply, IO updates and custom library additions
Add custom symbols/footprints for Keystone 4966 and AO4407A, and SOIC127P600X175-8N
footprint. Update sym-lib-table to reference new custom library.

Co-Authored-By: Claude Opus 4.7 (1M context) <noreply@anthropic.com>
Parts:
- removed C1, C5: 10uF, Capacitor_SMD:C_0805_2012Metric, symbol Device:C
- removed C2: 22uF, Capacitor_SMD:C_0805_2012Metric, symbol Device:C
- removed C3: 100nF, Capacitor_SMD:C_0603_1608Metric, symbol Device:C
- removed D2: MBR0530, Diode_SMD:D_SOD-123, symbol Device:D_Schottky
- removed FH3: 2A ATM, BatteryMonitorModule_Custom:FUSE_BK-6013, symbol Device:Fuse
- removed J2: OSTYK42102030, BatteryMonitorModule_Custom:OSTYK42102030, symbol Connector:Screw_Terminal_01x02
- removed L1: 4.7uH, BatteryMonitorModule_Custom:IND_BOURNS_SRR4028, symbol Device:L
- removed R25: 82k, Resistor_SMD:R_0603_1608Metric, symbol Device:R
- removed R26: 33k, Resistor_SMD:R_0603_1608Metric, symbol Device:R
- removed TP8: 5V, TestPoint:TestPoint_Pad_2.0x2.0mm, symbol Connector:TestPoint_Square
- removed TP9: 3.3V, TestPoint:TestPoint_Pad_2.0x2.0mm, symbol Connector:TestPoint_Square
- removed U3: AP63205WU-7, BatteryMonitorModule_Custom:AP63205WU-7_DIO, symbol AP63205WU-7:AP63205WU-7
- removed U4: TC2117-3.3VDBTR, Package_TO_SOT_SMD:SOT-223-3_TabPin2, symbol TC2117-3.3VDBTR:TC2117-3.3VDBTR
Other:
- note removed: "12->5V"
- note removed: "5V USB Bus -> Diode ->5V bus Nominally USB at 5.25 or lower won't pass unless no 12 V present. 12V -> 5V Regulator is pulled up to always enable in either 12 or usb connected This means if no 12V present enters LV protection Does not pull 5V low so 5VUSB will dominate."
- note removed: "5V->3.3 LDO"
