File: CAD/BatteryMonitorModule_V1/BatteryMonitorModule/BatteryMonitorModule.kicad_pcb (KiCad board)
At the start: 2 copper layers, 74.6 x 74.6 mm, 72 parts, among them J1 J_FAN, J2 QT06ADP83H0000G, J3 J_NFC, J4 J_PANEL, J5 J_UART, J6 Conn_ARM_JTAG_SWD_10, J7 USB-C, K1 G5Q-14-DC12, Q1 AO4407A, Q2 AO4407A, Q3 AO3400A, Q4 MMBT2222A, Q5 2N7002, SW1 BOOT0, SW2 NRST, U1 STM32C071K8T6, U2 AP63203WU-7, U3 INA226AQDGSRQ1

Commit message: PCB update
Parts:
- moved D3 101.0 mm to (53.9, 67.9), turned to 90 degrees
- moved D2 97.1 mm to (56.4, 67.9), turned to 90 degrees
- moved PE_GND1 96.6 mm to (67.3, 37.8), turned to -90 degrees
- moved LED1 92.4 mm to (68.1, 47.6), turned to -90 degrees
- moved C2 90.8 mm to (55.0, 74.0), turned to -90 degrees
- moved LED3 86.0 mm to (80.0, 48.2), turned to 90 degrees
- moved L1 85.0 mm to (61.2, 66.0), turned to 180 degrees
- moved U2 71.8 mm to (60.3, 73.0)
- moved R15 67.6 mm to (89.0, 50.2), turned to 90 degrees
- moved Q4 64.4 mm to (58.0, 79.0)
- moved LED2 62.5 mm to (84.0, 84.2), turned to 90 degrees
- moved Q3 60.2 mm to (57.9, 84.0)
- moved C3 58.0 mm to (65.0, 72.6), turned to -90 degrees
- moved D1 57.9 mm to (91.0, 83.0), turned to 180 degrees
- moved TP1 49.5 mm to (94.0, 46.0)
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Routing:
- net USB_D+: track 45.9 -> 0.00 mm
- net USB_D-: track 45.9 -> 0.00 mm
- net UART1_TX: track 10.5 -> 0.00 mm
- net UART1_RX: track 10.5 -> 0.00 mm
