File: CAD/BatteryMonitorModule_V1/BatteryMonitorModule/BatteryMonitorModule.kicad_sch (KiCad schematic)
At the start: 76 parts, among them J1 J_FAN, J2 QT06ADP83H0000G, J3 J_NFC, J4 J_PANEL, J5 J_UART, J6 Conn_ARM_JTAG_SWD_10, J7 USB-C, J8 J_PANEL, K1 G5Q-14-DC12, Q1 AO4407A, Q2 AO4407A, Q3 AO3400A, Q4 MMBT2222A, Q5 2N7002, SW1 BOOT0, SW2 NRST, U1 STM32C071K8T6, U2 AP63203WU-7, U3 INA226AQDGSRQ1

Commit message: found wiring error and fixed. Reved board from - to 1
Parts:
- C1, C3, C4, C7, C9: Digikey PN (none) -> 1276-1001-6-ND; MANUFACTURER (none) -> Samsung Electro-Mechanics; MPN (none) -> CL05B104KO5NNNC; Source (none) -> Digikey
- C2: Digikey PN (none) -> 1276-6454-6-ND; MANUFACTURER (none) -> Samsung Electro-Mechanics; MPN (none) -> CL21A106KAYNNNG; Source (none) -> Digikey
- C5, C6: Digikey PN (none) -> 1276-1100-6-ND; MANUFACTURER (none) -> Samsung Electro-Mechanics; MPN (none) -> CL21A226MQQNNNE; Source (none) -> Digikey
- C8: Digikey PN (none) -> 1276-1044-6-ND; MANUFACTURER (none) -> Samsung Electro-Mechanics; MPN (none) -> CL10A475KP8NNNC; Source (none) -> Digikey
- D1, D4: Digikey PN (none) -> 5399-1N4148WDKR-ND; MANUFACTURER (none) -> Shenzhen Slkormicro Semicon Co., Ltd.; MPN (none) -> 1N4148W; Source (none) -> Digikey
- D2, D3: Digikey PN (none) -> 5399-SS14DKR-ND; MANUFACTURER (none) -> Shenzhen Slkormicro Semicon Co., Ltd.; MPN (none) -> SS14; Source (none) -> Digikey
- F1, F2, F3: Digikey PN (none) -> BK-6013-ND; MANUFACTURER (none) -> MPD (Memory Protection Devices); MPN (none) -> BK-6013; Source (none) -> Digikey
- J1: Digikey PN (none) -> 455-B2B-XH-A-ND; MANUFACTURER (none) -> JST Sales America Inc.; MPN (none) -> B2B-XH-A; Source (none) -> Digikey
- J2: Digikey PN (none) -> 1818-QT06ADP83H0000G-ND; MANUFACTURER (none) -> Amphenol Anytek; MPN (none) -> QT06ADP83H0000G; Source (none) -> Digikey
- J3: Digikey PN (none) -> 455-B4B-XH-A-ND; MANUFACTURER (none) -> JST Sales America Inc.; MPN (none) -> B4B-XH-A; Source (none) -> Digikey
- J4, J5: Source (none) -> N/A; now not fitted
- J6: Digikey PN (none) -> N/A; MPN (none) -> Generic; Source (none) -> Alliexpress
- J7: Digikey PN (none) -> 2223-UJ20-C-H-G-SMT-1-P16-TRDKR-ND; MPN (none) -> UJ20-C-H-G-SMT-1-P16-TR; Source (none) -> Digikey
- J8: Source (none) -> Amazon
- K1: value G5Q-14-DC12 -> ALQ312; MANUFACTURER (none) -> Omron Electronics Inc-EMC Div; MPN (none) -> ALQ312; Source (none) -> Digikey
- L1: Digikey PN (none) -> SRR4028-3R3YTR-ND; MANUFACTURER (none) -> Bourns Inc.; MPN (none) -> SRR4028-3R3Y; Source (none) -> Digikey
- LED1, LED2, LED3: Digikey PN (none) -> 160-1435-6-ND; MANUFACTURER (none) -> Lite-On Inc.; MPN (none) -> LTST-C190KGKT; Source (none) -> Digikey
- PE_GND1: Digikey PN (none) -> 36-4966-ND; MANUFACTURER (none) -> Keystone Electronics; MPN (none) -> 4966; Source (none) -> Digikey
- Q1, Q2: value AO4407A -> SI4435FDY-T1-GE3; Digikey PN (none) -> SI4435FDY-T1-GE3DKR-ND; MANUFACTURER Alpha & Omega Semiconductor -> Vishay Siliconix; MPN (none) -> SI4435FDY-T1-GE3; Source (none) -> Digikey
- Q3: Digikey PN (none) -> 785-1000-2-ND; MANUFACTURER (none) -> Alpha & Omega Semiconductor; MPN (none) -> AO3400A; Source (none) -> Digikey
- Q4: Digikey PN (none) -> 5399-MMBT2222ADKR-ND; MANUFACTURER (none) -> Shenzhen Slkormicro Semicon Co., Ltd.; MPN (none) -> MMBT2222A; Source (none) -> Digikey
- Q5: Digikey PN (none) -> 5399-2N7002TR-ND; MANUFACTURER (none) -> Shenzhen Slkormicro Semicon Co., Ltd.; MPN (none) -> 2N7002; Source (none) -> Digikey
- R1, R11, R14, R19, R24, R9: Digikey PN (none) -> RMCF0402FT10K0DKR-ND; MANUFACTURER (none) -> Stackpole Electronics Inc; MPN (none) -> RMCF0402FT10K0; Source (none) -> Digikey
- R10: Digikey PN (none) -> 311-100KLRDKR-ND; MANUFACTURER (none) -> YAGEO; MPN (none) -> RC0402FR-07100KL; Source (none) -> Digikey
- R12, R17, R8: Digikey PN (none) -> 311-100LRDKR-ND; MANUFACTURER (none) -> YAGEO; MPN (none) -> RC0402FR-07100RL; Source (none) -> Digikey
- R13: value 10m -> 4m; Digikey PN (none) -> 4506-PEWF2512F4L00Q9CT-ND; MANUFACTURER (none) -> C&B/RESI; MPN (none) -> PEWF2512F4L00Q9; Source (none) -> Digikey
- R15: Digikey PN (none) -> 2019-RK73B1ETTP563JDKR-ND; MANUFACTURER (none) -> KOA Speer Electronics, Inc.; MPN (none) -> RK73B1ETTP563J; Source (none) -> Digikey
- R16: Digikey PN (none) -> RMCF0402FT68K0DKR-ND; MANUFACTURER (none) -> Stackpole Electronics Inc; MPN (none) -> RMCF0402FT68K0; Source (none) -> Digikey
- R18: Digikey PN (none) -> 311-1.00KLRDKR-ND; MANUFACTURER (none) -> YAGEO; MPN (none) -> RC0402FR-071KL; Source (none) -> Digikey
- R2, R20, R21, R22, R23, R25, R26, R3: Digikey PN (none) -> RMCF0402FT5K10DKR-ND; MANUFACTURER (none) -> Stackpole Electronics Inc; MPN (none) -> RMCF0402FT5K10; Source (none) -> Digikey
- R4, R5, R6, R7: Digikey PN (none) -> A138481CT-ND; MANUFACTURER (none) -> TE Connectivity Passive Product; MPN (none) -> RR03J62RTB
- RT1: Digikey PN (none) -> 445-174327-6-ND; MANUFACTURER (none) -> TDK; MPN (none) -> NTCG164BH103JT1; Source (none) -> Digikey
- SW1, SW2: Digikey PN (none) -> 450-1140-ND; MANUFACTURER (none) -> TE Connectivity ALCOSWITCH Switches; MPN (none) -> FSMSM; Source (none) -> Digikey
- TF1: Digikey PN (none) -> 317-RT184-ND; MANUFACTURER (none) -> Cantherm; MPN (none) -> RT184; Source (none) -> Digikey
- U1: Digikey PN (none) -> 497-STM32C071K8T6-ND; MANUFACTURER (none) -> STM; MPN (none) -> STM32C071K8T6; Source (none) -> Digikey
- U2: Digikey PN (none) -> AP63203WU-7DIDKR-ND; MANUFACTURER (none) -> Diodes Incorporated; MPN (none) -> AP63203WU-7; Source (none) -> Digikey
- U3: Digikey PN (none) -> 296-INA237AIDGSRCT-ND; MANUFACTURER (none) -> Texas Instruments; MPN (none) -> INA237AIDGSR; Source (none) -> Digikey
Connections:
- net USB_D+: now also U1.23 (PA12); no longer U1.22 (PA11)
- net USB_D-: now also U1.22 (PA11); no longer U1.23 (PA12)
