File: CAD/BatteryMonitorModule_V1/BatteryMonitorModule/BatteryMonitorModule.kicad_sch (KiCad schematic)
At the start: 76 parts, among them J1 J_FAN, J2 QT06ADP83H0000G, J3 J_NFC, J4 J_PANEL, J5 J_UART, J6 Conn_ARM_JTAG_SWD_10, J7 USB-C, J8 J_PANEL, K1 ALQ312, Q1 SI4435FDY-T1-GE3, Q2 SI4435FDY-T1-GE3, Q3 AO3400A, Q4 MMBT2222A, Q5 2N7002, SW1 BOOT0, SW2 NRST, U1 STM32C071K8T6, U2 AP63203WU-7, U3 INA226AQDGSRQ1

Commit message: INA238 driver + cdc_print + FLASH size reduction+ linker rename (#5)
* feat(ina238): driver + i2c_bus mutex/DMA + smoke task

- Driver: INA238 with INA237 compat (identical register map + scaling).
  ina238_probe() accepts either device ID and records the variant in
  dev->detected_device_id.
- Bus wrapper (Core/Src/i2c_bus.c): mutex for I2C1 sharing (INA238 +
  future PN532), DMA-completion semaphore, HAL callback overrides.
- CubeMX regen: I2C1 SMBus-slave -> I2C master, NoStretch=Disable
  (PN532-friendly), DMA1 ch1/ch2 TX/RX, ~338 kHz on PCLK1=48 MHz.
  SMBus HAL files dropped.
- Smoke task: bus scan, raw MFG/DEV ID dump, register-state dump after
  configure, 1 Hz sample loop with K1 relay toggle, per-line raw VSHUNT
  and VBUS register reads, runtime stack HWM.
- CDC robustness: TX buffer 64 -> 256, writer loops on short returns so
  multi-line bursts no longer drop trailing bytes.
- Stack tracking trio: runtime osThreadGetStackSpace HWM, static .su +
  objdump call-graph walk (scripts/stack_report.py + cmake stack_report
  target), pthread sentinel-fill UT helper (test/support/stack_measure).
- 37 host-side Ceedling tests pass; added :expect_any_args CMock plugin
  and pthread link flag.
- Schematic updated to INA238.

Bring-up status: I2C path proven -- chip IDs (0x5449/0x2381 = INA238)
and VBUS scaling both clean. VSHUNT register reads at the chip's
input-offset floor (~5 uV) regardless of current through R13; firmware
side fully validated, suspect a sense-pin solder issue on the
4-terminal shunt.

Co-Authored-By: Claude Opus 4.7 (1M context) <noreply@anthropic.com>

* feat(cdc_print): printf logger + libc retarget; -5 KB via int-only vfprintf

cdc_print module:
- Mutex-protected shared 256 B format buffer; any task can cdc_printf()
  without its own char[N] scratch. Mutex also serialises whole lines so
  two tasks can't interleave bytes mid-format.
- cdc_write blocks (loops + osDelay(1)) when the TX FIFO is full; drops
  silently if no host is connected.
-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
Parts:
- U3: value INA226AQDGSRQ1 -> INA238
Changed lines of the file:
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@@
 			)
 		)
-		(property "Value" "INA226AQDGSRQ1"
+		(property "Value" "INA238"
 			(at 217.678 156.464 0)
 			(show_name no)
